File: DemoGit.kicad_sch (KiCad schematic)
At the start: 16 parts, among them J1 USB_B_Micro, J2 Conn_Coaxial, SW1 SW_Push, U1 AP2112K-3.3, U2 RFM95W-915S2, U3 ATSAMD21G15A-A

Commit message: feat(sch): agrega display e-ink U4 al esquemático
Parts:
- added U4: Waveshare_epaper, Display_7Segment:7SegmentLED_LTS6760_LTS6780, symbol E_Ink_Display:E_ink_display
Changed lines of the file:
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@@
+	)
+	(symbol
+		(lib_id "E_Ink_Display:E_ink_display")
+		(at 168.91 144.78 0)
+		(unit 1)
+		(body_style 1)
+		(exclude_from_sim no)
+		(in_bom yes)
+		(on_board yes)
+		(in_pos_files yes)
+		(dnp no)
+		(fields_autoplaced yes)
+		(property "Reference" "U4"
+			(at 171.0533 137.16 0)
+			(show_name no)
+			(do_not_autoplace no)
+			(effects
+				(font
+					(size 1.27 1.27)
+				)
+				(justify left)
+			)
+		)
+		(property "Value" "Waveshare_epaper"
+			(at 171.0533 139.7 0)
+			(show_name no)
+			(do_not_autoplace no)
+			(effects
+				(font
+					(size 1.27 1.27)
+				)
+				(justify left)
+			)
+		)
+		(property "Footprint" "Display_7Segment:7SegmentLED_LTS6760_LTS6780"
+			(at 168.91 144.78 0)
+			(hide yes)
+			(show_name no)
+			(do_not_autoplace no)
+			(effects
+				(font
+					(size 1.27 1.27)
+				)
+			)
+		)
+		(property "Datasheet" ""
+			(at 168.91 144.78 0)
+			(hide yes)
+			(show_name no)
+			(do_not_autoplace no)
+			(effects
+				(font
+					(size 1.27 1.27)
+				)
+			)
+		)
+		(property "Description" ""
+			(at 168.91 144.78 0)
+			(hide yes)
+			(show_name no)
+			(do_not_autoplace no)
+			(effects
+				(font
+					(size 1.27 1.27)
+				)
+			)
+		)
+		(pin "3"
+		)
+		(pin "1"
+		)
+		(pin "4"
+		)
+		(pin "8"
+		)
+		(pin "2"
+		)
+		(pin "7"
+		)
+		(pin "5"
+		)
+		(pin "6"
+		)
+		(instances
+			(project "DemoGit"
+				(path "/47592ec3-9c69-46c5-a8c2-f085c078fc65"
+					(reference "U4")
+					(unit 1)
+				)
+			)
+		)
 	)
 	(symbol
